Commit message: Builds via colcon

File: src/robot_description/urdf/robot.urdf (robot description, URDF)
Before this commit: robot simple_robot, 4 links, 3 joints
Links:
- removed link base_footprint
- added link camera_link, mass 0.1; collision box size=0.01 0.01 0.01; visual box size=0.01 0.01 0.01
- added link frontleft_wheel, mass 0.2; collision cylinder length=0.03 radius=0.0325; visual cylinder length=0.03 radius=0.0325
- added link frontright_wheel, mass 0.2; collision cylinder length=0.03 radius=0.0325; visual cylinder length=0.03 radius=0.0325
- added link lidar, mass 0.1; collision cylinder length=0.018 radius=0.033; visual cylinder length=0.018 radius=0.033
- added link top_floor, mass 0.3; collision box size=0.15 0.085 0.038; visual box size=0.15 0.085 0.038
- link base_link: mass 1.0 -> 1.5; geometry collision box size=0.28 0.23 0.07; visual box size=0.28 0.23 0.07
- link left_wheel: mass 0.1 -> 0.2; geometry collision cylinder length=0.03 radius=0.0325; visual cylinder length=0.03 radius=0.0325
- link right_wheel: mass 0.1 -> 0.2; geometry collision cylinder length=0.03 radius=0.0325; visual cylinder length=0.03 radius=0.0325
Joints:
- removed joint base_footprint_joint
- removed joint left_wheel_joint
- removed joint right_wheel_joint
- added joint base_frontleft_wheel_joint: type continuous, parent base_link, child frontleft_wheel, origin xyz=0.1075 0.13 0 rpy=0 0 0, axis 0 1 0
- added joint base_frontright_wheel_joint: type continuous, parent base_link, child frontright_wheel, origin xyz=0.1075 -0.13 0 rpy=0 0 0, axis 0 1 0
- added joint base_left_wheel_joint: type continuous, parent base_link, child left_wheel, origin xyz=-0.1075 0.13 0 rpy=0 0 0, axis 0 1 0
- added joint base_lidar_joint: type fixed, parent base_link, child lidar, origin xyz=0 0 0.103 rpy=0 0 0
- added joint base_right_wheel_joint: type continuous, parent base_link, child right_wheel, origin xyz=-0.1075 -0.13 0 rpy=0 0 0, axis 0 1 0
- added joint base_top_floor_joint: type fixed, parent base_link, child top_floor, origin xyz=0 0 0.085 rpy=0 0 0
- added joint camera_joint: type fixed, parent top_floor, child camera_link, origin xyz=0.08 0 0.01 rpy=0 0 0

File: src/robot_description/urdf/robot.urdf.xacro (robot description, xacro)
@@ -1,136 +1,109 @@
 <?xml version="1.0"?>
-<robot name="robot_car" xmlns:xacro="http://www.ros.org/wiki/xacro">
-  <!-- Arguments -->
-  <xacro:arg name="use_ros2_control" default="true" />
-  <!-- Include Sensors -->
-  <xacro:include filename="$(find robot_description)/urdf/sensors/rplidar.urdf.xacro" />
-  <!-- RPLIDAR Gazebo plugin -->
-  <gazebo reference="rplidar_link">
-    <sensor type="ray" name="rplidar">
-      <pose>0 0 0 0 0 0</pose>
-      <visualize>true</visualize>
-      <update_rate>10</update_rate>
-      <ray>
-        <scan>
-          <horizontal>
-            <samples>360</samples>
-            <resolution>1.0</resolution>
-            <min_angle>0.0</min_angle>
-            <max_angle>6.28319</max_angle>
-          </horizontal>
-        </scan>
-        <range>
-          <min>0.15</min>
-          <max>12.0</max>
-          <resolution>0.01</resolution>
-        </range>
-        <noise>
-          <type>gaussian</type>
-          <mean>0.0</mean>
-          <stddev>0.01</stddev>
-        </noise>
-      </ray>
-      <plugin name="gazebo_ros_rplidar_controller" filename="libgazebo_ros_ray_sensor.so">
-        <ros>
-          <namespace>/</namespace>
-          <remapping>~/out:=scan</remapping>
-        </ros>
-        <output_type>sensor_msgs/msg/LaserScan</output_type>
-        <frame_name>rplidar_link</frame_name>
-      </plugin>
-    </sensor>
-  </gazebo>
-  <!-- Sensor platform for mounting sensors -->
-  <link name="sensor_platform">
-    <visual>
-      <geometry>
-        <box size="0.15 0.085 0.038"/>
-      </geometry>
-      <material name="sensor_white"/>
-    </visual>
-    <collision>
-      <geometry>
-        <box size="0.15 0.085 0.038"/>
-      </geometry>
-    </collision>
-    <inertial>
-      <mass value="0.1"/>
-      <inertia ixx="0.0001" ixy="0" ixz="0" iyy="0.0001" iyz="0" izz="0.0001"/>
-    </inertial>
-  </link>
-  <!-- Joint to connect sensor platform to base -->
-  <joint name="sensor_platform_joint" type="fixed">
-    <parent link="base_link"/>
-    <child link="sensor_platform"/>
-    <origin xyz="0 0 0.05" rpy="0 0 0"/>
-  </joint>
-  <!-- Joint to connect RPLIDAR to sensor platform -->
-  <joint name="laser_joint" type="fixed">
-    <parent link="sensor_platform"/>
-    <child link="rplidar_link"/>
-    <origin xyz="0 0 0.03" rpy="0 0 0"/>
-  </joint>
-  <!-- Materials -->
-  <material name="sensor_white">
-    <color rgba="0.9 0.9 0.9 1"/>
-  </material>
-  <!-- Camera parameters -->
-  <xacro:property name="camera_width" value="0.05" />
-  <xacro:property name="camera_height" value="0.03" />
-  <xacro:property name="camera_depth" value="0.05" />
-  <xacro:property name="camera_x" value="0.1" />  <!-- Position in front of the robot -->
-  <xacro:property name="camera_y" value="0.0" />
-  <xacro:property name="camera_z" value="0.05" />
-  <xacro:property name="camera_fps" value="30" />
-  <xacro:property name="camera_hfov" value="1.0472" />  <!-- 60 degrees in radians -->
+<robot name="zeta" xmlns:xacro="http://www.ros.org/wiki/xacro">
   <!-- Constants -->
-  <xacro:property name="PI" value="3.1415926535897931" />
-  <!-- Robot dimensions (in meters) - Matching dojo_robot.urdf.xacro -->
-  <xacro:property name="base_length" value="0.23" />
-  <xacro:property name="base_width" value="0.28" />
-  <xacro:property name="base_height" value="0.07" />
+  <xacro:property name="M_PI" value="3.1415926535897931" />
+  <xacro:property name="M_PI_2" value="1.5707963267948966" />
+  <!-- Robot Parameters -->
+  <xacro:property name="base_x" value="0.28" />
+  <xacro:property name="base_y" value="0.23" />
+  <xacro:property name="base_z" value="0.07" />
   <xacro:property name="wheel_radius" value="0.0325" />
   <xacro:property name="wheel_width" value="0.03" />
   <xacro:property name="wheel_separation" value="0.26" />
-  <xacro:property name="wheel_base" value="0.215" />
-  <xacro:property name="caster_radius" value="0.01" />
   <!-- Materials -->
-  <material name="dojo_green">
-    <color rgba="0.2 0.8 0.2 1"/>
-  </material>
-  <material name="wheel_grey">
-    <color rgba="0.4 0.4 0.4 1"/>
-  </material>
-  <!-- Base footprint (for navigation) -->
-  <link name="base_footprint"/>
+  <material name="grey">
+    <color rgba="0.7 0.7 0.7 1"/>
+  </material>
+  <material name="green">
+    <color rgba="0 0.6 0 1"/>
+  </material>
+  <material name="white">
+    <color rgba="1 1 1 1"/>
+  </material>
+  <material name="black">
+    <color rgba="0.1 0.1 0.1 1"/>
+  </material>
+  <!-- Gazebo materials -->
+  <gazebo reference="base_link">
+    <material>Gazebo/Green</material>
+  </gazebo>
+  <gazebo reference="top_floor">
+    <material>Gazebo/Green</material>
+  </gazebo>
+  <gazebo reference="lidar">
+    <material>Gazebo/White</material>
+  </gazebo>
+  <gazebo reference="left_wheel">
+    <material>Gazebo/Grey</material>
+  </gazebo>
+  <gazebo reference="right_wheel">
+    <material>Gazebo/Grey</material>
+  </gazebo>
+  <gazebo reference="frontright_wheel">
+    <material>Gazebo/Grey</material>
+  </gazebo>
+  <gazebo reference="frontleft_wheel">
+    <material>Gazebo/Grey</material>
+  </gazebo>
   <!-- Base link -->
-  <!-- Base -->
   <link name="base_link">
     <visual>
-      <origin xyz="0 0 ${base_height/2}" rpy="0 0 0"/>
-      <geometry>
-        <box size="${base_length} ${base_width} ${base_height}"/>
-      </geometry>
-      <material name="blue"/>
-    </visual>
-    <collision>
-      <origin xyz="0 0 ${base_height/2}" rpy="0 0 0"/>
-      <geometry>
-        <box size="${base_length} ${base_width} ${base_height}"/>
-      </geometry>
-    </collision>
-  </link>
-  <!-- Wheels -->
+      <geometry>
+        <box size="${base_x} ${base_y} ${base_z}"/>
+      </geometry>
+      <origin xyz="0 0 0.035" rpy="0 0 0"/>
+      <material name="green"/>
+    </visual>
+    <collision>
+      <geometry>
+        <box size="${base_x} ${base_y} ${base_z}"/>
+      </geometry>
+      <origin xyz="0 0 0.035" rpy="0 0 0"/>
+    </collision>
+    <inertial>
+      <mass value="1.5"/>
+      <inertia ixx="0.003" ixy="0.0" ixz="0.0"
+               iyy="0.002" iyz="0.0"
+               izz="0.003"/>
+    </inertial>
+  </link>
+  <!-- Top floor -->
+  <link name="top_floor">
+    <visual>
+      <geometry>
+        <box size="0.15 0.085 0.038"/>
+      </geometry>
+      <origin xyz="0 0 0" rpy="0 0 0"/>
+      <material name="green"/>
+    </visual>
+    <collision>
+      <geometry>
+        <box size="0.15 0.085 0.038"/>
+      </geometry>
+      <origin xyz="0 0 0" rpy="0 0 0"/>
+    </collision>
+    <inertial>
+      <mass value="0.3"/>
+      <inertia ixx="0.0001" ixy="0.0" ixz="0.0"
+               iyy="0.0001" iyz="0.0"
+               izz="0.0001"/>
+    </inertial>
+  </link>
+  <!-- Joint between base and top floor -->
+  <joint name="base_to_top_floor" type="fixed">
+    <parent link="base_link"/>
+    <child link="top_floor"/>
+    <origin xyz="0 0 0.069" rpy="0 0 0"/>
+  </joint>
+  <!-- Wheel Macro -->
   <xacro:macro name="wheel" params="prefix x y z">
     <link name="${prefix}_wheel">
       <visual>
-        <origin xyz="0 0 0" rpy="${PI/2} 0 0"/>
         <geometry>
           <cylinder radius="${wheel_radius}" length="${wheel_width}"/>
         </geometry>
-        <material name="black"/>
+        <material name="grey"/>
       </visual>
       <collision>
-        <origin xyz="0 0 0" rpy="${PI/2} 0 0"/>
         <geometry>
           <cylinder radius="${wheel_radius}" length="${wheel_width}"/>
@@ -139,7 +112,5 @@
       <inertial>
         <mass value="0.1"/>
-        <inertia ixx="0.0005" ixy="0" ixz="0"
-                 iyy="0.0005" iyz="0"
-                 izz="0.0001"/>
+        <inertia ixx="0.0001" ixy="0.0" ixz="0.0" iyy="0.0001" iyz="0.0" izz="0.0001"/>
       </inertial>
     </link>
@@ -147,156 +118,92 @@
       <parent link="base_link"/>
       <child link="${prefix}_wheel"/>
-      <origin xyz="${x} ${y} ${z}" rpy="0 0 0"/>
+      <origin xyz="${x} ${y} ${z}" rpy="${M_PI_2} 0 0"/>
       <axis xyz="0 1 0"/>
-      <limit effort="100" velocity="100"/>
-      <dynamics damping="0.1" friction="0.5"/>
     </joint>
   </xacro:macro>
-  <!-- Casters -->
-  <xacro:macro name="caster" params="prefix x y z">
-    <link name="${prefix}_caster">
-      <visual>
-        <origin xyz="0 0 0" rpy="0 0 0"/>
-        <geometry>
-          <sphere radius="${caster_radius}"/>
-        </geometry>
-        <material name="gray"/>
-      </visual>
-      <collision>
-        <origin xyz="0 0 0" rpy="0 0 0"/>
-        <geometry>
-          <sphere radius="${caster_radius}"/>
-        </geometry>
-      </collision>
-      <inertial>
-        <mass value="0.01"/>
-        <inertia ixx="0.00001" ixy="0" ixz="0"
-                 iyy="0.00001" iyz="0"
-                 izz="0.00001"/>
-      </inertial>
-    </link>
-    <joint name="${prefix}_caster_joint" type="fixed">
-      <parent link="base_link"/>
-      <child link="${prefix}_caster"/>
-      <origin xyz="${x} ${y} ${z}" rpy="0 0 0"/>
-    </joint>
-  </xacro:macro>
-  <!-- Create wheels and casters -->
-  <xacro:wheel prefix="left" x="0" y="${wheel_separation/2}" z="0"/>
-  <xacro:wheel prefix="right" x="0" y="-${wheel_separation/2}" z="0"/>
-  <xacro:caster prefix="front" x="${base_length/4}" y="0" z="-${base_height/2}"/>
-  <xacro:caster prefix="back" x="-${base_length/4}" y="0" z="-${base_height/2}"/>
-  <!-- Base link joint -->
-  <joint name="base_footprint_joint" type="fixed">
-    <parent link="base_footprint"/>
-    <child link="base_link"/>
-    <origin xyz="0 0 ${wheel_radius}" rpy="0 0 0"/>
+  <!-- Create wheels -->
+  <xacro:wheel prefix="left" x="0" y="${base_y/2 + 0.01}" z="0"/>
+  <xacro:wheel prefix="right" x="0" y="-${base_y/2 - 0.01}" z="0"/>
+  <xacro:wheel prefix="frontleft" x="${base_x/2}" y="${base_y/2 + 0.01}" z="0"/>
+  <xacro:wheel prefix="frontright" x="${base_x/2}" y="-${base_y/2 - 0.01}" z="0"/>
+  <!-- Lidar -->
+  <link name="lidar">
+    <visual>
+      <geometry>
+        <cylinder radius="0.03" length="0.05"/>
+      </geometry>
+      <origin xyz="0 0 0" rpy="0 0 0"/>
+      <material name="white"/>
+    </visual>
+    <collision>
+      <geometry>
+        <cylinder radius="0.03" length="0.05"/>
+      </geometry>
+      <origin xyz="0 0 0" rpy="0 0 0"/>
+    </collision>
+    <inertial>
+      <mass value="0.1"/>
+      <inertia ixx="0.0001" ixy="0.0" ixz="0.0" iyy="0.0001" iyz="0.0" izz="0.0001"/>
+    </inertial>
+  </link>
+  <joint name="lidar_joint" type="fixed">
+    <parent link="top_floor"/>
+    <child link="lidar"/>
+    <origin xyz="0 0 0.04" rpy="0 0 0"/>
   </joint>
-  <!-- ROS 2 Control -->
-  <xacro:if value="$(arg use_ros2_control)">
-    <!-- Gazebo ROS control -->
-    <gazebo>
-      <plugin filename="libgazebo_ros2_control.so" name="gazebo_ros2_control">
-        <parameters>/robot_description</parameters>
-        <controller_manager_node_name>controller_manager</controller_manager_node_name>
-      </plugin>
-    </gazebo>
-    <!-- ROS 2 Control -->
-    <ros2_control name="GazeboSystem" type="system">
-      <hardware>
-        <plugin>gazebo_ros2_control/GazeboSystem</plugin>
-      </hardware>
-      <joint name="left_wheel_joint">
-        <command_interface name="velocity"/>
-        <state_interface name="position"/>
-        <state_interface name="velocity"/>
-      </joint>
-      <joint name="right_wheel_joint">
-        <command_interface name="velocity"/>
-        <state_interface name="position"/>
-        <state_interface name="velocity"/>
-      </joint>
-    </ros2_control>
-  </xacro:if>
-  <!-- Camera link -->
-  <link name="camera_link">
-    <visual>
-      <origin xyz="${camera_x} ${camera_y} ${camera_z}" rpy="0 0 0"/>
-      <geometry>
-        <box size="${camera_width} ${camera_height} ${camera_depth}"/>
-      </geometry>
-      <material name="sensor_white"/>
-    </visual>
-    <collision>
-      <origin xyz="${camera_x} ${camera_y} ${camera_z}" rpy="0 0 0"/>
-      <geometry>
-        <box size="${camera_width} ${camera_height} ${camera_depth}"/>
-      </geometry>
-    </collision>
-  </link>
-  <!-- Camera joint -->
+  <!-- Camera -->
+  <link name="camera">
+    <visual>
+      <geometry>
+        <box size="0.02 0.04 0.03"/>
+      </geometry>
+      <origin xyz="0 0 0" rpy="0 0 0"/>
+      <material name="black">
+        <color rgba="0.1 0.1 0.1 1"/>
+      </material>
+    </visual>
+    <collision>
+      <geometry>
+        <box size="0.02 0.04 0.03"/>
+      </geometry>
+      <origin xyz="0 0 0" rpy="0 0 0"/>
+    </collision>
+    <inertial>
+      <mass value="0.05"/>
+      <inertia ixx="0.00001" ixy="0.0" ixz="0.0" iyy="0.00001" iyz="0.0" izz="0.00001"/>
+    </inertial>
+  </link>
   <joint name="camera_joint" type="fixed">
-    <parent link="base_link"/>
-    <child link="camera_link"/>
-    <origin xyz="0 0 0" rpy="0 0 0"/>
+    <parent link="top_floor"/>
+    <child link="camera"/>
+    <origin xyz="0.08 0 0.01" rpy="0 0 0"/>
   </joint>
-  <!-- Camera sensor -->
-  <gazebo reference="camera_link">
-    <sensor type="camera" name="camera1">
-      <update_rate>${camera_fps}</update_rate>
-      <camera name="front">
-        <horizontal_fov>${camera_hfov}</horizontal_fov>
-        <image>
-          <width>640</width>
-          <height>480</height>
-          <format>R8G8B8</format>
-        </image>
-        <clip>
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
Commit message: cleanup

File: src/robot_description/urdf/robot.urdf (robot description, URDF)
Before this commit: robot zeta, 8 links, 7 joints
Links:
- link frontleft_wheel: mass 0.2 -> 0.1
- link frontright_wheel: mass 0.2 -> 0.1
- link left_wheel: mass 0.2 -> 0.1
- link lidar: geometry collision cylinder length=0.05 radius=0.03; visual cylinder length=0.05 radius=0.03
- link right_wheel: mass 0.2 -> 0.1

File: src/robot_description/urdf/robot.urdf.xacro (robot description, xacro)
@@ -91,8 +91,8 @@
   </link>
   <!-- Joint between base and top floor -->
-  <joint name="base_to_top_floor" type="fixed">
+  <joint name="base_top_floor_joint" type="fixed">
     <parent link="base_link"/>
     <child link="top_floor"/>
-    <origin xyz="0 0 0.069" rpy="0 0 0"/>
+    <origin xyz="0 0 0.085" rpy="0 0 0"/>
   </joint>
   <!-- Wheel Macro -->
@@ -115,16 +115,16 @@
       </inertial>
     </link>
-    <joint name="${prefix}_wheel_joint" type="continuous">
+    <joint name="base_${prefix}_wheel_joint" type="continuous">
       <parent link="base_link"/>
       <child link="${prefix}_wheel"/>
-      <origin xyz="${x} ${y} ${z}" rpy="${M_PI_2} 0 0"/>
+      <origin xyz="${x} ${y} ${z}" rpy="0 0 0"/>
       <axis xyz="0 1 0"/>
     </joint>
   </xacro:macro>
   <!-- Create wheels -->
-  <xacro:wheel prefix="left" x="0" y="${base_y/2 + 0.01}" z="0"/>
-  <xacro:wheel prefix="right" x="0" y="-${base_y/2 - 0.01}" z="0"/>
-  <xacro:wheel prefix="frontleft" x="${base_x/2}" y="${base_y/2 + 0.01}" z="0"/>
-  <xacro:wheel prefix="frontright" x="${base_x/2}" y="-${base_y/2 - 0.01}" z="0"/>
+  <xacro:wheel prefix="left" x="-0.1075" y="0.13" z="0"/>
+  <xacro:wheel prefix="right" x="-0.1075" y="-0.13" z="0"/>
+  <xacro:wheel prefix="frontleft" x="0.1075" y="0.13" z="0"/>
+  <xacro:wheel prefix="frontright" x="0.1075" y="-0.13" z="0"/>
   <!-- Lidar -->
   <link name="lidar">
@@ -147,28 +147,26 @@
     </inertial>
   </link>
-  <joint name="lidar_joint" type="fixed">
-    <parent link="top_floor"/>
+  <joint name="base_lidar_joint" type="fixed">
+    <parent link="base_link"/>
     <child link="lidar"/>
-    <origin xyz="0 0 0.04" rpy="0 0 0"/>
+    <origin xyz="0 0 0.103" rpy="0 0 0"/>
   </joint>
   <!-- Camera -->
-  <link name="camera">
-    <visual>
-      <geometry>
-        <box size="0.02 0.04 0.03"/>
-      </geometry>
-      <origin xyz="0 0 0" rpy="0 0 0"/>
-      <material name="black">
-        <color rgba="0.1 0.1 0.1 1"/>
-      </material>
-    </visual>
-    <collision>
-      <geometry>
-        <box size="0.02 0.04 0.03"/>
-      </geometry>
-      <origin xyz="0 0 0" rpy="0 0 0"/>
-    </collision>
-    <inertial>
-      <mass value="0.05"/>
+  <link name="camera_link">
+    <visual>
+      <geometry>
+        <box size="0.01 0.01 0.01"/>
+      </geometry>
+      <origin xyz="0 0 0" rpy="0 0 0"/>
+      <material name="black"/>
+    </visual>
+    <collision>
+      <geometry>
+        <box size="0.01 0.01 0.01"/>
+      </geometry>
+      <origin xyz="0 0 0" rpy="0 0 0"/>
+    </collision>
+    <inertial>
+      <mass value="0.1"/>
       <inertia ixx="0.00001" ixy="0.0" ixz="0.0" iyy="0.00001" iyz="0.0" izz="0.00001"/>
     </inertial>
@@ -176,8 +174,72 @@
   <joint name="camera_joint" type="fixed">
     <parent link="top_floor"/>
-    <child link="camera"/>
+    <child link="camera_link"/>
     <origin xyz="0.08 0 0.01" rpy="0 0 0"/>
   </joint>
-  <!-- Gazebo Plugins -->
+  <!-- Gazebo Camera Sensor -->
+  <gazebo reference="camera_link">
+    <sensor type="camera" name="camera1">
+      <update_rate>30.0</update_rate>
+      <camera name="front">
+        <horizontal_fov>1.3962634</horizontal_fov>
+        <image>
+          <width>640</width>
+          <height>480</height>
+          <format>R8G8B8</format>
+        </image>
+        <clip>
+          <near>0.1</near>
+          <far>100</far>
+        </clip>
+      </camera>
+      <plugin name="camera_controller" filename="libgazebo_ros_camera.so">
+        <ros>
+          <namespace>/</namespace>
+        </ros>
+        <camera_name>camera</camera_name>
+        <frame_name>camera_link</frame_name>
+        <hack_baseline>0.07</hack_baseline>
+      </plugin>
+      <always_on>true</always_on>
+      <update_rate>30.0</update_rate>
+      <visualize>true</visualize>
+    </sensor>
+  </gazebo>
+  <!-- Gazebo LiDAR Sensor -->
+  <gazebo reference="lidar">
+    <sensor type="ray" name="lidar_sensor">
+      <pose>0 0 0 0 0 0</pose>
+      <visualize>true</visualize>
+      <update_rate>10</update_rate>
+      <ray>
+        <scan>
+          <horizontal>
+            <samples>360</samples>
+            <resolution>1</resolution>
+            <min_angle>-3.14159</min_angle>
+            <max_angle>3.14159</max_angle>
+          </horizontal>
+        </scan>
+        <range>
+          <min>0.1</min>
+          <max>12.0</max>
+          <resolution>0.01</resolution>
+        </range>
+        <noise>
+          <type>gaussian</type>
+          <mean>0.0</mean>
+          <stddev>0.01</stddev>
+        </noise>
+      </ray>
+      <plugin name="gazebo_ros_lidar" filename="libgazebo_ros_ray_sensor.so">
+        <ros>
+          <namespace>/</namespace>
+        </ros>
+        <output_type>sensor_msgs/LaserScan</output_type>
+        <frame_name>lidar</frame_name>
+      </plugin>
+    </sensor>
+  </gazebo>
+  <!-- Gazebo Differential Drive Plugin -->
   <gazebo>
     <plugin name="differential_drive_controller" filename="libgazebo_ros_diff_drive.so">
@@ -185,6 +247,8 @@
         <namespace>/</namespace>
       </ros>
-      <left_joint>left_wheel_joint</left_joint>
-      <right_joint>right_wheel_joint</right_joint>
+      <left_joint>base_left_wheel_joint</left_joint>
+      <left_joint>base_frontleft_wheel_joint</left_joint>
+      <right_joint>base_right_wheel_joint</right_joint>
+      <right_joint>base_frontright_wheel_joint</right_joint>
       <wheel_separation>${wheel_separation}</wheel_separation>
       <wheel_diameter>${2 * wheel_radius}</wheel_diameter>
@@ -195,15 +259,8 @@
       <publish_odom>true</publish_odom>
       <publish_odom_tf>true</publish_odom_tf>
-      <publish_wheel_tf>false</publish_wheel_tf>
+      <publish_wheel_tf>true</publish_wheel_tf>
+      <max_wheel_torque>0.5</max_wheel_torque>
+      <max_wheel_acceleration>1.0</max_wheel_acceleration>
     </plugin>
-    <plugin name="camera_controller" filename="libgazebo_ros_camera.so">
-      <alwaysOn>true</alwaysOn>
-      <updateRate>30.0</updateRate>
-      <cameraName>camera</cameraName>
-      <frameName>camera</frameName>
-      <imageTopicName>image_raw</imageTopicName>
-      <cameraInfoTopicName>camera_info</cameraInfoTopicName>
-      <hackBaseline>0.07</hackBaseline>
-    </plugin>
   </gazebo>
 </robot>
