Commit message: feat: Implement ROSbot XL simulation, control, and autonomous navigation with supporting diagnostic tools.

File: src/rosbot_xl_description/urdf/gazebo.urdf.xacro (robot description, xacro)
@@ -43,4 +43,6 @@
         <visualize>false</visualize>
         <enable_metrics>false</enable_metrics>
+        <plugin filename="gz-sim-imu-system" name="gz::sim::systems::Imu">
+        </plugin>
         <frame_id>imu_link</frame_id>
         <ignition_frame_id>imu_link</ignition_frame_id>

File: src/rosbot_xl_description/urdf/rosbot_xl.urdf.xacro (robot description, xacro)
@@ -2,5 +2,5 @@
 <robot name="rosbot_xl" xmlns:xacro="http://www.ros.org/wiki/xacro">
   <xacro:arg name="mecanum" default="false" />
-  <xacro:arg name="lidar_model" default="slamtec_rplidar_s1" />
+  <xacro:arg name="lidar_model" default="slamtec_rplidar" />
   <xacro:arg name="camera_model" default="intel_realsense_d435" />
   <xacro:arg name="include_camera_mount" default="false" />
@@ -28,5 +28,5 @@
   <xacro:property name="lidar_model" value="$(arg lidar_model)" />
   <xacro:property name="lidar_parent_link" value="cover_link" />
-  <xacro:property name="lidar_xyz" value="0.02 0.0 0.0" />
+  <xacro:property name="lidar_xyz" value="0.02 0.0 0.2" />
   <xacro:property name="lidar_rpy" value="0.0 0.0 0.0" />
   <xacro:if value="${lidar_model == 'slamtec_rplidar_s1'}">

File: src/rosbot_xl_description/urdf/rosbot_xl_macro.urdf.xacro (robot description, xacro)
@@ -61,5 +61,5 @@
         <xacro:if value="${use_sim}">
           <xacro:if value="${simulation_engine == 'ignition-gazebo'}">
-            <plugin>ign_ros2_control/IgnitionSystem</plugin>
+            <plugin>gz_ros2_control/GazeboSimSystem</plugin>
           </xacro:if>
           <xacro:if value="${simulation_engine == 'webots'}">
@@ -121,4 +121,6 @@
         <xacro:gazebo.controller config_file="${controller_config_file}" namespace="${namespace}" />
         <xacro:gazebo.imu reference_frame="imu_link" namespace="${namespace}" />
+        <!-- Gazebo Drive Plugins removed to avoid conflict with ros2_control -->
+        <!-- ros2_control handles drive and odometry via MecanumDriveController or DiffDriveController -->
       </xacro:if>
       <xacro:if value="${simulation_engine == 'webots'}">

File: src/rosbot_xl_description/urdf/wheel.urdf.xacro (robot description, xacro)
@@ -84,6 +84,12 @@
               <ode>
                 <mu>1.0</mu>
-                <mu2>0.0</mu2>
-                <fdir1 ignition:expressed_in="base_link">${fdir}</fdir1>
+                <xacro:if value="${mecanum}">
+                  <mu2>0.0</mu2>
+                  <fdir1 ignition:expressed_in="base_link">${fdir}</fdir1>
+                </xacro:if>
+                <xacro:unless value="${mecanum}">
+                  <mu2>1.0</mu2>
+                  <fdir1 ignition:expressed_in="base_link">1 0 0</fdir1>
+                </xacro:unless>
               </ode>
             </friction>
