Commit message: feat: Integrate twist mux, add semantic object visualization, update Gazebo bridging and lidar position, and enhance dynamic world loading with camera topic remapping.

File: src/rosbot_xl_description/urdf/rosbot_xl.urdf.xacro (robot description, xacro)
@@ -28,5 +28,5 @@
   <xacro:property name="lidar_model" value="$(arg lidar_model)" />
   <xacro:property name="lidar_parent_link" value="cover_link" />
-  <xacro:property name="lidar_xyz" value="0.02 0.0 0.2" />
+  <xacro:property name="lidar_xyz" value="0.02 0.0 0.0" />
   <xacro:property name="lidar_rpy" value="0.0 0.0 0.0" />
   <xacro:if value="${lidar_model == 'slamtec_rplidar_s1'}">
